File: schematics/petpuller.kicad_pcb (KiCad board)
At the start: 2 copper layers, 99.7 x 99.7 mm, 47 parts, among them J1 Heater, J2 Motor Conn, J3 Thermistor, J4 Power Input, J5 TXRX, J6 AdditionalAnalog, J7 Heater, J8 Heater, Q1 IRFZ34N, Q2 BC547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

Commit message: fixes
Parts:
- added C2: 100uF, Capacitor_THT:CP_Radial_D8.0mm_P2.50mm, F.Cu at (162.6, 25.4)
- added C3: 100uF, Capacitor_THT:CP_Radial_D8.0mm_P2.50mm, F.Cu at (102.9, 34.3)
- added R20: 10K, Resistor_SMD:R_0805_2012Metric_Pad1.20x1.40mm_HandSolder, B.Cu at (152.4, 56.5)
- added R21: 10K, Resistor_SMD:R_0805_2012Metric_Pad1.20x1.40mm_HandSolder, B.Cu at (154.9, 56.5)
- added R9: 10K, Resistor_SMD:R_0805_2012Metric_Pad1.20x1.40mm_HandSolder, B.Cu at (149.9, 56.5)
- moved Q1 5.43 mm to (175.9, 58.4), turned to 0 degrees
- moved Q4 5.43 mm to (175.9, 47.0), turned to 0 degrees
- moved Q6 5.43 mm to (175.9, 35.6), turned to 0 degrees
Connections:
- Q1 pad 1: Net-(J1-Pad2) -> Net-(Q1-Pad1)
- Q1 pad 2: Net-(Q1-Pad2) -> Net-(J1-Pad2)
- Q2 pad 1: Net-(Q1-Pad2) -> Net-(Q1-Pad1)
- Q4 pad 1: Net-(J7-Pad2) -> Net-(Q3-Pad1)
- Q4 pad 2: Net-(Q3-Pad1) -> Net-(J7-Pad2)
- Q6 pad 1: Net-(J8-Pad2) -> Net-(Q5-Pad1)
- Q6 pad 2: Net-(Q5-Pad1) -> Net-(J8-Pad2)
- R1 pad 2: Net-(Q1-Pad2) -> Net-(Q1-Pad1)
- R11 pad 1: Net-(Q1-Pad2) -> Net-(Q1-Pad1)
Routing:
- net +5V: track 182.4 -> 227.1 mm, vias 2 -> 3
- net Net-(Q1-Pad1): track 0.00 -> 17.5 mm
- net Net-(Q1-Pad2): track 16.7 -> 0.00 mm
- net Net-(J8-Pad2): track 7.25 -> 13.1 mm
- net Net-(J7-Pad2): track 7.25 -> 13.1 mm
- net Net-(J1-Pad2): track 7.25 -> 13.1 mm
- net heater: track 22.2 -> 24.3 mm
- net fan: track 28.8 -> 31.0 mm
- net additionalPwm: track 35.9 -> 38.1 mm
- net Net-(Q3-Pad1): track 16.6 -> 17.4 mm
